File: mucol_pcb/mucol_pcb.kicad_sch (KiCad schematic)
At the start: 0 parts

Commit message: ESP32 schematic
ESP32 şematiği çıktı, footprintler eklenmesi seçilmesi lazım.
Parts:
- added C1, C11, C14, C5, C8, C9: 22u, symbol Device:C_Small
- added C10, C12, C13, C15, C16, C2, C6: 100n, symbol Device:C_Small
- added C3, C4: 4u7, symbol Device:C_Small
- added C7: 1000u/25V, symbol Device:C_Polarized_Small
- added D1: LED_RGBA, symbol Device:LED_RGBA
- added D2: LL4148, Diode_SMD:D_MiniMELF, symbol Diode:LL4148
- added D3, D4: LED, LED_SMD:LED_0402_1005Metric, symbol Device:LED
- added F1: 1A, symbol Device:Polyfuse_Small
- added F2: Fuse, symbol Device:Fuse
- added FB1: FB, symbol Device:FerriteBead_Small
- added H1, H2, H3, H4: MountingHole_Pad, symbol Mechanical:MountingHole_Pad
- added J1: USB_C_Receptacle_USB2.0_16P, Connector_USB:USB_C_Receptacle_Palconn_UTC16-G, symbol Connector:USB_C_Receptacle_USB2.0_16P
- added J2: Screw_Terminal_01x02, symbol Connector:Screw_Terminal_01x02
- added J3: Screw_Terminal_01x08, symbol Connector:Screw_Terminal_01x08
- added J4: Conn_01x04, Connector_JST:JST_VH_B4P-VH_1x04_P3.96mm_Vertical, symbol Connector_Generic:Conn_01x04
- added J5: Screw_Terminal_01x03, symbol Connector:Screw_Terminal_01x03
- added J6: Conn_02x05_Odd_Even, symbol Connector_Generic:Conn_02x05_Odd_Even
- added K1: RT314A05, Relay_THT:Relay_SPDT_Schrack-RT1-16A-FormC_RM5mm, symbol Relay:RT314A05
- added Q1, Q2: UMH3N, Package_TO_SOT_SMD:SOT-363_SC-70-6, symbol Transistor_BJT:UMH3N
- added Q3: BC817, Package_TO_SOT_SMD:SOT-23, symbol Transistor_BJT:BC817
- added R1, R19, R7: 10K, symbol Device:R_Small
- added R10, R6, R8, R9: 1K, symbol Device:R_Small
- added R11, R12: 4k7, symbol Device:R_Small
- added R13: 10k, symbol Device:R_Small
- added R14: 1k, symbol Device:R_Small
- added R15, R16, R17, R18, R4, R5: 22R, symbol Device:R_Small
- added R2, R3: 5.1K, symbol Device:R_Small
- added SW1: SW_SPST, symbol Switch:SW_SPST
- added U1: LM1117MP-3.3, Package_TO_SOT_SMD:SOT-223-3_TabPin2, symbol Regulator_Linear:LM1117MP-3.3
- added U2: CP2104, Package_DFN_QFN:QFN-24-1EP_4x4mm_P0.5mm_EP2.6x2.6mm, symbol Interface_USB:CP2104
- added U3: USBLC6-2P6, Package_TO_SOT_SMD:SOT-666, symbol Power_Protection:USBLC6-2P6
- added U4: 74HC245, symbol 74xx:74HC245
- added U5: ESP32-WROOM-32U, RF_Module:ESP32-WROOM-32U, symbol RF_Module:ESP32-WROOM-32U
- added U6: Si7021-A20, Package_DFN_QFN:DFN-6-1EP_3x3mm_P1mm_EP1.5x2.4mm, symbol Sensor_Humidity:Si7021-A20
Connections:
- new net: J1.A5 (CC1), R3.1
- new net: J1.A6 (D+), J1.B6 (D+), U3.3 (I/O2)
- new net: J1.A7 (D-), J1.B7 (D-), U3.1 (I/O1)
- new net: J1.B5 (CC2), R2.1
- new net: C3.1, U2.16 (VPP)
- new net: R5.1, U2.20 (RXD)
- new net: R4.1, U2.21 (TXD)
- new net: R1.2, U2.9 (~{RST})
- new net: F1.1, FB1.2
- new net: J5.2 (Pin_2), K1.11
- new net: J5.1 (Pin_1), K1.12
- new net: J5.3 (Pin_3), K1.14
- new net: D2.2 (A), D3.1 (K), K1.A2, Q3.3 (C)
- new net: Q3.1 (B), R13.2, R14.1
- new net: D1.3 (BK), R10.2
- new net: D1.1 (RK), R8.2
- new net: C7.1, F2.1, J2.1 (Pin_1)
- new net: R15.1, U4.18 (B0)
- new net: J3.3 (Pin_3), R15.2
- new net: R18.1, U4.15 (B3)
- new net: R17.1, U4.16 (B2)
- new net: R16.1, U4.17 (B1)
- new net: D1.2 (GK), R9.2
- new net: J3.5 (Pin_5), R17.2
- new net: J3.4 (Pin_4), R16.2
- new net: D4.1 (K), R6.1
- new net: J3.6 (Pin_6), R18.2
- new net: F2.2, J3.1 (Pin_1), J3.2 (Pin_2)
- new net +3.3V: C11.1, C12.1, C14.1, C15.1, C9.1, D1.4 (A), D4.2 (A), J4.2 (Pin_2), J6.1 (Pin_1), J6.2 (Pin_2), R11.2, R12.2, R19.1, R7.1, U1.2 (VO), U5.2 (VDD), U6.5 (VDD)
- new net +3.3VA: C5.1, C6.1, R1.1, U2.5 (VIO), U2.6 (VDD)
- new net +5V: C1.1, C13.1, C2.1, C4.1, C8.1, D2.1 (K), D3.2 (A), F1.2, K1.A1, U1.3 (VI), U2.7 (REGIN), U2.8 (VBUS), U3.5 (VBUS), U4.1 (A->B), U4.20 (VCC)
- new net +5VP: FB1.1, J1.A4 (VBUS), J1.A9 (VBUS), J1.B4 (VBUS), J1.B9 (VBUS)
- new net DTR: Q1.1 (E1), Q2.2 (B1), U2.23 (~{DTR})
- new net D_L: U2.3 (D+), U3.4 (I/O2)
- new net D_N: U2.4 (D-), U3.6 (I/O1)
- new net EN: C16.1, Q2.1 (E1), R19.2, U5.3 (EN)
- new net GND: C1.2, C10.2, C11.2, C12.2, C13.2, C14.2, C15.2, C16.2, C2.2, C3.2, C4.2, C5.2, C6.2, C7.2, C8.2, C9.2, H1.1, H2.1, H3.1, H4.1, J1.A1 (GND), J1.A12 (GND), J1.B1 (GND), J1.B12 (GND), J1.S1 (SHIELD), J2.2 (Pin_2), J4.1 (Pin_1), J6.10 (Pin_10), J6.9 (Pin_9), Q3.2 (E), R13.1, R2.2, R3.2, R6.2, SW1.1 (A), U1.1 (GND), U2.2 (GND), U2.25 (GND), U3.2 (GND), U4.10 (GND), U4.19 (CE), U4.6 (A4), U4.7 (A5), U4.8 (A6), U4.9 (A7), U5.1 (GND), U5.15 (GND), U5.38 (GND), U5.39 (GND), U6.2 (GND), U6.7 (PAD)
- new net GPIO26: J6.3 (Pin_3), U5.11 (IO26)
- new net GPIO27: J6.5 (Pin_5), U5.12 (IO27)
- new net GPIO32: J6.7 (Pin_7), U5.8 (IO32)
- new net GPIO33: J6.4 (Pin_4), U5.9 (IO33)
- new net GPIO34: J6.6 (Pin_6), U5.6 (IO34)
- new net GPIO35: J6.8 (Pin_8), U5.7 (IO35)
- new net IO0: Q1.6 (C1), U5.25 (IO0)
- new net LEDSTR1: U4.2 (A0), U5.27 (IO16)
- new net LEDSTR2: U4.3 (A1), U5.28 (IO17)
- new net LEDSTR3: U4.4 (A2), U5.30 (IO18)
- new net LEDSTR4: U4.5 (A3), U5.31 (IO19)
- new net LED_B: R10.1, U5.23 (IO15)
- new net LED_G: R9.1, U5.13 (IO14)
- new net LED_R: R8.1, U5.16 (IO13)
- new net RELAY: R14.2, U5.10 (IO25)
- new net RTS: Q1.2 (B1), Q2.6 (C1), U2.19 (~{RTS})
- new net RX: R4.2, U5.35 (TXD0/IO1)
- new net SCL: J4.4 (Pin_4), R11.1, U5.37 (IO23), U6.6 (SCL)
- new net SDA: J4.3 (Pin_3), R12.1, U5.36 (IO22), U6.1 (SDA)
- new net SW: C10.1, R7.2, SW1.2 (B), U5.33 (IO21)
- new net TX: R5.2, U5.34 (RXD0/IO3)
- no-connect marks 0 -> 6
Other:
- note added: "GND"
- note added: "RXD"
- note added: "SCL"
- note added: "SDA"
- note added: "TXD"
- note added: "VDD"

Commit message: Şematik Kod
Other:
- note added: "Bu bakılacak"
- moved on the sheet: C14, C15, C16, J6, R19, U5
