File: prototipV1/prototipV1.kicad_sch (KiCad schematic)
At the start: 19 parts, among them U1 ESP32_KIT, U2 L7812, U3 LM2596S-ADJ

Commit message: güncelleme
Parts:
- added D7, D8: D_Schottky, symbol Device:D_Schottky
Connections:
- net at C2.1, C3.1, U2.3 (OUT): now also D8.2 (A); no longer U3.1 (VIN)
- new net 2SBAT: D7.1 (K), D8.1 (K), U3.1 (VIN)
